Commit message: gazebo simulation added

File: robotis_op3_description/_urdf/robotis_op3.gazebo.xacro (robot description, xacro)
@@ -8,6 +8,4 @@
   <!-- body link -->
   <gazebo reference="body_link">
-    <mu1>0.2</mu1>
-    <mu2>0.2</mu2>
     <material>Gazebo/White</material>
     <selfCollide>false</selfCollide>
@@ -15,71 +13,50 @@
   <!-- left leg links -->
   <gazebo reference="l_hip_yaw_link">
-    <mu1>0.2</mu1>
-    <mu2>0.2</mu2>
     <material>Gazebo/White</material>
     <selfCollide>false</selfCollide>
   </gazebo>
   <gazebo reference="l_hip_roll_link">
-    <mu1>0.2</mu1>
-    <mu2>0.2</mu2>
     <material>Gazebo/White</material>
     <selfCollide>false</selfCollide>
   </gazebo>
   <gazebo reference="l_hip_pitch_link">
-    <mu1>0.2</mu1>
-    <mu2>0.2</mu2>
     <material>Gazebo/White</material>
     <selfCollide>false</selfCollide>
   </gazebo>
   <gazebo reference="l_knee_link">
-    <mu1>0.2</mu1>
-    <mu2>0.2</mu2>
     <material>Gazebo/White</material>
     <selfCollide>false</selfCollide>
   </gazebo>
   <gazebo reference="l_ank_pitch_link">
-    <mu1>0.2</mu1>
-    <mu2>0.2</mu2>
     <material>Gazebo/White</material>
     <selfCollide>false</selfCollide>
   </gazebo>
   <gazebo reference="l_ank_roll_link">
-    <kp>100000.0</kp>
-    <kd>100.0</kd>
-    <mu1>1.5</mu1>
-    <mu2>1.5</mu2>
-    <fdir1>1 0 0</fdir1>
-    <maxVel>1.0</maxVel>
+    <mu1>9000</mu1>
+    <mu2>9000</mu2>
+    <kp>1000000.0</kp>
+    <kd>10.0</kd>
     <minDepth>0.001</minDepth>
+    <maxContacts>1</maxContacts>
     <material>Gazebo/White</material>
   </gazebo>
   <!-- right leg links -->
   <gazebo reference="r_hip_yaw_link">
-    <mu1>0.2</mu1>
-    <mu2>0.2</mu2>
     <material>Gazebo/White</material>
     <selfCollide>false</selfCollide>
   </gazebo>
   <gazebo reference="r_hip_roll_link">
-    <mu1>0.2</mu1>
-    <mu2>0.2</mu2>
     <material>Gazebo/White</material>
     <selfCollide>false</selfCollide>
   </gazebo>
   <gazebo reference="r_hip_pitch_link">
-    <mu1>0.2</mu1>
-    <mu2>0.2</mu2>
     <material>Gazebo/White</material>
     <selfCollide>false</selfCollide>
   </gazebo>
   <gazebo reference="r_knee_link">
-    <mu1>0.2</mu1>
-    <mu2>0.2</mu2>
     <material>Gazebo/White</material>
     <selfCollide>false</selfCollide>
   </gazebo>
   <gazebo reference="r_ank_pitch_link">
-    <mu1>0.2</mu1>
-    <mu2>0.2</mu2>
     <material>Gazebo/White</material>
     <selfCollide>false</selfCollide>
@@ -87,58 +64,40 @@
   <gazebo reference="r_ank_roll_link">
     <mu1>9000</mu1>
-    <kp>100000.0</kp>
-    <kd>100.0</kd>
-    <mu1>1.5</mu1>
-    <mu2>1.5</mu2>
-    <fdir1>1 0 0</fdir1>
-    <maxVel>1.0</maxVel>
+    <mu2>9000</mu2>
+    <kp>1000000.0</kp>
+    <kd>10.0</kd>
     <minDepth>0.001</minDepth>
+    <maxContacts>1</maxContacts>
     <material>Gazebo/White</material>
   </gazebo>
   <gazebo reference="r_sho_pitch_link">
-    <mu1>0.2</mu1>
-    <mu2>0.2</mu2>
     <material>Gazebo/White</material>
     <selfCollide>false</selfCollide>
   </gazebo>
   <gazebo reference="r_sho_roll_link">
-    <mu1>0.2</mu1>
-    <mu2>0.2</mu2>
     <material>Gazebo/White</material>
     <selfCollide>false</selfCollide>
   </gazebo>
   <gazebo reference="r_el_link">
-    <mu1>0.2</mu1>
-    <mu2>0.2</mu2>
     <material>Gazebo/White</material>
     <selfCollide>false</selfCollide>
   </gazebo>
   <gazebo reference="l_sho_pitch_link">
-    <mu1>0.2</mu1>
-    <mu2>0.2</mu2>
     <material>Gazebo/White</material>
     <selfCollide>false</selfCollide>
   </gazebo>
   <gazebo reference="l_sho_roll_link">
-    <mu1>0.2</mu1>
-    <mu2>0.2</mu2>
     <material>Gazebo/White</material>
     <selfCollide>false</selfCollide>
   </gazebo>
   <gazebo reference="l_el_link">
-    <mu1>0.2</mu1>
-    <mu2>0.2</mu2>
     <material>Gazebo/White</material>
     <selfCollide>false</selfCollide>
   </gazebo>
   <gazebo reference="head_pan_link">
-    <mu1>0.2</mu1>
-    <mu2>0.2</mu2>
     <material>Gazebo/White</material>
     <selfCollide>false</selfCollide>
   </gazebo>
   <gazebo reference="head_tilt_link">
-    <mu1>0.2</mu1>
-    <mu2>0.2</mu2>
     <material>Gazebo/White</material>
     <selfCollide>false</selfCollide>
@@ -227,5 +186,4 @@
 -->
   <!-- head camera -->
-<!--
   <gazebo reference="cam_link">
     <sensor name='camera' type='camera'>
@@ -261,5 +219,4 @@
     </sensor>
   </gazebo>
--->
   <!-- imu sensor -->
 <!--

File: robotis_op3_description/_urdf/robotis_op3.structure.head.xacro (robot description, xacro)
@@ -12,5 +12,5 @@
     <origin xyz="-0.001 0.0 0.1365" rpy="0 0 0" />
     <axis xyz="0 0 1" />
-    <limit effort="1000" velocity="100" lower="${-pi*0.9}" upper="${pi*0.9}" />
+    <limit effort="1000" velocity="100" lower="${-pi*0.6}" upper="${pi*0.6}" />
     <dynamics damping="0.1" friction="0.0" />
   </joint>
@@ -34,5 +34,5 @@
     <origin xyz="0.010 0.019 0.0285" rpy="0 0 0" />
     <axis xyz="0 -1 0" />
-    <limit effort="1000" velocity="100" lower="${-pi*0.9}" upper="${pi*0.9}" />
+    <limit effort="1000" velocity="100" lower="${-pi*0.6}" upper="${pi*0.6}" />
     <dynamics damping="0.1" friction="0.0" />
   </joint>

File: robotis_op3_description/_urdf/robotis_op3.structure.larm.xacro (robot description, xacro)
@@ -12,5 +12,5 @@
     <origin xyz="-0.001 0.06 0.111" rpy="0 0 0" />
     <axis xyz="0 1 0" />
-    <limit effort="1000" velocity="100" lower="${-pi*0.9}" upper="${pi*0.9}" />
+    <limit effort="1000" velocity="100" lower="${-pi*0.6}" upper="${pi*0.6}" />
     <dynamics damping="0.1" friction="0.0" />
   </joint>
@@ -34,5 +34,5 @@
     <origin xyz="0.019 0.0285 -0.010" rpy="0 0 0" />
     <axis xyz="-1 0 0" />
-    <limit effort="1000" velocity="100" lower="${-pi*0.9}" upper="${pi*0.9}" />
+    <limit effort="1000" velocity="100" lower="${-pi*0.6}" upper="${pi*0.6}" />
     <dynamics damping="0.1" friction="0.0" />
   </joint>
@@ -56,5 +56,5 @@
     <origin xyz="0.0 0.0904 -0.0001" rpy="0 0 0" />
     <axis xyz="1 0 0" />
-    <limit effort="1000" velocity="100" lower="${-pi*0.9}" upper="${pi*0.9}" />
+    <limit effort="1000" velocity="100" lower="${-pi*0.6}" upper="${pi*0.6}" />
     <dynamics damping="0.1" friction="0.0" />
   </joint>

File: robotis_op3_description/_urdf/robotis_op3.structure.lleg.xacro (robot description, xacro)
@@ -12,5 +12,5 @@
     <origin xyz="0.0 0.035 0.0" rpy="0 0 0" />
     <axis xyz="0 0 -1" />
-    <limit effort="1000" velocity="100" lower="${-pi*0.9}" upper="${pi*0.9}" />
+    <limit effort="1000" velocity="100" lower="${-pi*0.6}" upper="${pi*0.6}" />
     <dynamics damping="0.1" friction="0.0" />
   </joint>
@@ -34,5 +34,5 @@
     <origin xyz="-0.024 0.0 -0.0285" rpy="0 0 0" />
     <axis xyz="-1 0 0" />
-    <limit effort="1000" velocity="100" lower="${-pi*0.9}" upper="${pi*0.9}" />
+    <limit effort="1000" velocity="100" lower="${-pi*0.6}" upper="${pi*0.6}" />
     <dynamics damping="0.1" friction="0.0" />
   </joint>
@@ -56,5 +56,5 @@
     <origin xyz="0.0241 0.019 0.0" rpy="0 0 0" />
     <axis xyz="0 1 0" />
-    <limit effort="1000" velocity="100" lower="${-pi*0.9}" upper="${pi*0.9}" />
+    <limit effort="1000" velocity="100" lower="${-pi*0.6}" upper="${pi*0.6}" />
     <dynamics damping="0.1" friction="0.0" />
   </joint>
@@ -78,5 +78,5 @@
     <origin xyz="0.0 0.0 -0.11015" rpy="0 0 0" />
     <axis xyz="0 1 0" />
-    <limit effort="1000" velocity="100" lower="${-pi*0.9}" upper="${pi*0.9}" />
+    <limit effort="1000" velocity="100" lower="${-pi*0.6}" upper="${pi*0.6}" />
     <dynamics damping="0.1" friction="0.0" />
   </joint>
@@ -100,5 +100,5 @@
     <origin xyz="0 0 -0.110" rpy="0 0 0" />
     <axis xyz="0 -1 0" />
-    <limit effort="1000" velocity="100" lower="${-pi*0.9}" upper="${pi*0.9}" />
+    <limit effort="1000" velocity="100" lower="${-pi*0.6}" upper="${pi*0.6}" />
     <dynamics damping="0.1" friction="0.0" />
   </joint>
@@ -122,5 +122,5 @@
     <origin xyz="-0.0241 -0.019 0" rpy="0 0 0" />
     <axis xyz="1 0 0" />
-    <limit effort="1000" velocity="100" lower="${-pi*0.9}" upper="${pi*0.9}" />
+    <limit effort="1000" velocity="100" lower="${-pi*0.6}" upper="${pi*0.6}" />
     <dynamics damping="0.1" friction="0.0" />
   </joint>

File: robotis_op3_description/_urdf/robotis_op3.structure.rarm.xacro (robot description, xacro)
@@ -12,5 +12,5 @@
     <origin xyz="-0.001 -0.06 0.111" rpy="0 0 0" />
     <axis xyz="0 -1 0" />
-    <limit effort="1000" velocity="100" lower="${-pi*0.9}" upper="${pi*0.9}" />
+    <limit effort="1000" velocity="100" lower="${-pi*0.6}" upper="${pi*0.6}" />
     <dynamics damping="0.1" friction="0.0" />
   </joint>
@@ -34,5 +34,5 @@
     <origin xyz="0.019 -0.0285 -0.010" rpy="0 0 0" />
     <axis xyz="-1 0 0" />
-    <limit effort="1000" velocity="100" lower="${-pi*0.9}" upper="${pi*0.9}" />
+    <limit effort="1000" velocity="100" lower="${-pi*0.6}" upper="${pi*0.6}" />
     <dynamics damping="0.1" friction="0.0" />
   </joint>
@@ -56,5 +56,5 @@
     <origin xyz="0.0 -0.0904 -0.0001" rpy="0 0 0" />
     <axis xyz="1 0 0" />
-    <limit effort="1000" velocity="100" lower="${-pi*0.9}" upper="${pi*0.9}" />
+    <limit effort="1000" velocity="100" lower="${-pi*0.6}" upper="${pi*0.6}" />
     <dynamics damping="0.1" friction="0.0" />
   </joint>

File: robotis_op3_description/_urdf/robotis_op3.structure.rleg.xacro (robot description, xacro)
@@ -12,5 +12,5 @@
     <origin xyz="0.0 -0.035 0.0" rpy="0 0 0" />
     <axis xyz="0 0 -1" />
-    <limit effort="1000" velocity="100" lower="${-pi*0.9}" upper="${pi*0.9}" />
+    <limit effort="1000" velocity="100" lower="${-pi*0.6}" upper="${pi*0.6}" />
     <dynamics damping="0.1" friction="0.0" />
   </joint>
@@ -34,5 +34,5 @@
     <origin xyz="-0.024 0.0 -0.0285" rpy="0 0 0" />
     <axis xyz="-1 0 0" />
-    <limit effort="1000" velocity="100" lower="${-pi*0.9}" upper="${pi*0.9}" />
+    <limit effort="1000" velocity="100" lower="${-pi*0.6}" upper="${pi*0.6}" />
     <dynamics damping="0.1" friction="0.0" />
   </joint>
@@ -56,5 +56,5 @@
     <origin xyz="0.0241 -0.019 0.0" rpy="0 0 0" />
     <axis xyz="0 -1 0" />
-    <limit effort="1000" velocity="100" lower="${-pi*0.9}" upper="${pi*0.9}" />
+    <limit effort="1000" velocity="100" lower="${-pi*0.6}" upper="${pi*0.6}" />
     <dynamics damping="0.1" friction="0.0" />
   </joint>
@@ -78,5 +78,5 @@
     <origin xyz="0.0 0.0 -0.11015" rpy="0 0 0" />
     <axis xyz="0 -1 0" />
-    <limit effort="1000" velocity="100" lower="${-pi*0.9}" upper="${pi*0.9}" />
+    <limit effort="1000" velocity="100" lower="${-pi*0.6}" upper="${pi*0.6}" />
     <dynamics damping="0.1" friction="0.0" />
   </joint>
@@ -100,5 +100,5 @@
     <origin xyz="0 0 -0.110" rpy="0 0 0" />
     <axis xyz="0 1 0" />
-    <limit effort="1000" velocity="100" lower="${-pi*0.9}" upper="${pi*0.9}" />
+    <limit effort="1000" velocity="100" lower="${-pi*0.6}" upper="${pi*0.6}" />
     <dynamics damping="0.1" friction="0.0" />
   </joint>
@@ -122,5 +122,5 @@
     <origin xyz="-0.0241 0.019 0" rpy="0 0 0" />
     <axis xyz="1 0 0" />
-    <limit effort="1000" velocity="100" lower="${-pi*0.9}" upper="${pi*0.9}" />
+    <limit effort="1000" velocity="100" lower="${-pi*0.6}" upper="${pi*0.6}" />
     <dynamics damping="0.1" friction="0.0" />
   </joint>

File: robotis_op3_description/_urdf/robotis_op3.urdf.xacro (robot description, xacro)
@@ -17,20 +17,4 @@
   <xacro:add_sim_harness harnessed_link="body_link"/>
   -->
-<!--
-  <link name="world">
-  </link>
-  <joint name="world_fixed" type="fixed">
-    <origin xyz="0 0 0" rpy="0 0 0"/>
-    <parent link="world"/>
-    <child link="base"/>
-  </joint>
-  <link name="base">
-  </link>
-  <joint name="base_fixed" type="fixed">
-    <origin xyz="0 0 0" rpy="0 0 0"/>
-    <parent link="base"/>
-    <child link="body_link"/>
-  </joint>
--->
   <!-- body link -->
   <link name="body_link">
@@ -45,11 +29,17 @@
     </inertial>
   </link>
-  <!-- leg link -->
+  <!-- leg links -->
+  <!--
   <xacro:robotis_op3_l_leg parent="body_link" />
   <xacro:robotis_op3_r_leg parent="body_link" />
-  <!-- arm link -->
+  -->
+  <!-- leg links -->
+  <!--
   <xacro:robotis_op3_l_arm parent="body_link" />
   <xacro:robotis_op3_r_arm parent="body_link" />
+  -->
   <!-- head links -->
+  <!--
   <xacro:robotis_op3_head parent="body_link" />
+  -->
 </robot>
