Commit message: gazebo camera imu added

File: robotis_op3_description/urdf/robotis_op3.gazebo.xacro (robot description, xacro)
@@ -227,6 +227,5 @@
 -->
   <!-- head camera -->
-<!--
-  <gazebo reference="cam_link">
+  <gazebo reference="cam_gazebo_link">
     <sensor name='camera' type='camera'>
       <pose>-0.050000 -0.010000 0.000000 -1.5708 0.000000 -3.141592</pose>
@@ -261,18 +260,23 @@
     </sensor>
   </gazebo>
--->
   <!-- imu sensor -->
-<!--
-  <gazebo>
-    <plugin filename="libhector_gazebo_ros_imu.so" name="gazebo_ros_imu">
-      <bodyName>body_link</bodyName>
-      <updateRate>50</updateRate>
-      <serviceName>/robotis_op3/imu_service</serviceName>
-      <topicName>/robotis_op3/imu</topicName>
-      <gaussianNoise>0</gaussianNoise>
-      <xyzOffset>0 0 0</xyzOffset>
-      <rpyOffset>0 0 -0.703220730592</rpyOffset>
-    </plugin>
-  </gazebo>
--->
+  <gazebo reference="body_link">
+    <gravity>true</gravity>
+    <sensor name="imu_sensor" type="imu">
+      <always_on>true</always_on>
+      <update_rate>100</update_rate>
+      <visualize>true</visualize>
+      <topic>__default_topic__</topic>
+      <plugin filename="libgazebo_ros_imu_sensor.so" name="imu_plugin">
+        <topicName>robotis_op3/imu</topicName>
+        <bodyName>imu_link</bodyName>
+        <updateRateHZ>10.0</updateRateHZ>
+        <gaussianNoise>0.0</gaussianNoise>
+        <xyzOffset>0 0 0</xyzOffset>
+        <rpyOffset>0 0 0</rpyOffset>
+        <frameName>imu_link</frameName>
+      </plugin>
+      <pose>0 0 0 0 0 0</pose>
+    </sensor>
+  </gazebo>
 </robot>

File: robotis_op3_description/urdf/robotis_op3.structure.head.xacro (robot description, xacro)
@@ -56,7 +56,15 @@
     <child link="cam_link"/>
   </joint>
+  <joint name="cam_gazebo" type="fixed">
+    <origin xyz="0.01425 -0.019 0.04975" rpy="0 0 0"/>
+    <parent link="head_tilt_link"/>
+    <child link="cam_gazebo_link"/>
+  </joint>
   <!-- camera link -->
   <link name="cam_link">
   </link>
+  <!-- camera link -->
+  <link name="cam_gazebo_link">
+  </link>
   </xacro:macro>
 </robot>
