Commit message: refactoring to release

File: robotis_op3_description/urdf/robotis_op3.visuals.xacro (robot description, xacro)
@@ -8,5 +8,5 @@
     <origin xyz="0 0 0" rpy="0 0 0" />
     <geometry>
-      <mesh filename="package://robotis_op3_description/stl/body.stl"  scale="0.001 0.001 0.001"/>
+      <mesh filename="package://robotis_op3_description/meshes/body.stl"  scale="0.001 0.001 0.001"/>
     </geometry>
     <material name="Grey">
@@ -18,5 +18,5 @@
     <origin xyz="0 0 0" rpy="0 0 0" />
     <geometry>
-      <mesh filename="package://robotis_op3_description/stl/rl1.stl"  scale="0.001 0.001 0.001"/>
+      <mesh filename="package://robotis_op3_description/meshes/rl1.stl"  scale="0.001 0.001 0.001"/>
     </geometry>
     <material name="Grey">
@@ -28,5 +28,5 @@
     <origin xyz="0 0 0" rpy="0 0 0" />
     <geometry>
-      <mesh filename="package://robotis_op3_description/stl/rl2.stl"  scale="0.001 0.001 0.001"/>
+      <mesh filename="package://robotis_op3_description/meshes/rl2.stl"  scale="0.001 0.001 0.001"/>
     </geometry>
     <material name="Grey">
@@ -38,5 +38,5 @@
     <origin xyz="0 0 0" rpy="0 0 0" />
     <geometry>
-      <mesh filename="package://robotis_op3_description/stl/rl3.stl"  scale="0.001 0.001 0.001"/>
+      <mesh filename="package://robotis_op3_description/meshes/rl3.stl"  scale="0.001 0.001 0.001"/>
     </geometry>
     <material name="Grey">
@@ -48,5 +48,5 @@
     <origin xyz="0 0 0" rpy="0 0 0" />
     <geometry>
-      <mesh filename="package://robotis_op3_description/stl/rl4.stl"  scale="0.001 0.001 0.001"/>
+      <mesh filename="package://robotis_op3_description/meshes/rl4.stl"  scale="0.001 0.001 0.001"/>
     </geometry>
     <material name="Grey">
@@ -58,5 +58,5 @@
     <origin xyz="0 0 0" rpy="0 0 0" />
     <geometry>
-      <mesh filename="package://robotis_op3_description/stl/rl5.stl"  scale="0.001 0.001 0.001"/>
+      <mesh filename="package://robotis_op3_description/meshes/rl5.stl"  scale="0.001 0.001 0.001"/>
     </geometry>
     <material name="Grey">
@@ -68,5 +68,5 @@
     <origin xyz="0 0 0" rpy="0 0 0" />
     <geometry>
-      <mesh filename="package://robotis_op3_description/stl/rl6.stl"  scale="0.001 0.001 0.001"/>
+      <mesh filename="package://robotis_op3_description/meshes/rl6.stl"  scale="0.001 0.001 0.001"/>
     </geometry>
     <material name="Grey">
@@ -78,5 +78,5 @@
     <origin xyz="0 0 0" rpy="0 0 0" />
     <geometry>
-      <mesh filename="package://robotis_op3_description/stl/ll1.stl"  scale="0.001 0.001 0.001"/>
+      <mesh filename="package://robotis_op3_description/meshes/ll1.stl"  scale="0.001 0.001 0.001"/>
     </geometry>
     <material name="Grey">
@@ -88,5 +88,5 @@
     <origin xyz="0 0 0" rpy="0 0 0" />
     <geometry>
-      <mesh filename="package://robotis_op3_description/stl/ll2.stl"  scale="0.001 0.001 0.001"/>
+      <mesh filename="package://robotis_op3_description/meshes/ll2.stl"  scale="0.001 0.001 0.001"/>
     </geometry>
     <material name="Grey">
@@ -98,5 +98,5 @@
     <origin xyz="0 0 0" rpy="0 0 0" />
     <geometry>
-      <mesh filename="package://robotis_op3_description/stl/ll3.stl"  scale="0.001 0.001 0.001"/>
+      <mesh filename="package://robotis_op3_description/meshes/ll3.stl"  scale="0.001 0.001 0.001"/>
     </geometry>
     <material name="Grey">
@@ -108,5 +108,5 @@
     <origin xyz="0 0 0" rpy="0 0 0" />
     <geometry>
-      <mesh filename="package://robotis_op3_description/stl/ll4.stl"  scale="0.001 0.001 0.001"/>
+      <mesh filename="package://robotis_op3_description/meshes/ll4.stl"  scale="0.001 0.001 0.001"/>
     </geometry>
     <material name="Grey">
@@ -118,5 +118,5 @@
     <origin xyz="0 0 0" rpy="0 0 0" />
     <geometry>
-      <mesh filename="package://robotis_op3_description/stl/ll5.stl"  scale="0.001 0.001 0.001"/>
+      <mesh filename="package://robotis_op3_description/meshes/ll5.stl"  scale="0.001 0.001 0.001"/>
     </geometry>
     <material name="Grey">
@@ -128,5 +128,5 @@
     <origin xyz="0 0 0" rpy="0 0 0" />
     <geometry>
-      <mesh filename="package://robotis_op3_description/stl/ll6.stl"  scale="0.001 0.001 0.001"/>
+      <mesh filename="package://robotis_op3_description/meshes/ll6.stl"  scale="0.001 0.001 0.001"/>
     </geometry>
     <material name="Grey">
@@ -138,5 +138,5 @@
     <origin xyz="0 0 0" rpy="0 0 0" />
     <geometry>
-      <mesh filename="package://robotis_op3_description/stl/ra1.stl"  scale="0.001 0.001 0.001"/>
+      <mesh filename="package://robotis_op3_description/meshes/ra1.stl"  scale="0.001 0.001 0.001"/>
     </geometry>
     <material name="Grey">
@@ -148,5 +148,5 @@
     <origin xyz="0 0 0" rpy="0 0 0" />
     <geometry>
-      <mesh filename="package://robotis_op3_description/stl/ra2.stl"  scale="0.001 0.001 0.001"/>
+      <mesh filename="package://robotis_op3_description/meshes/ra2.stl"  scale="0.001 0.001 0.001"/>
     </geometry>
     <material name="Grey">
@@ -158,5 +158,5 @@
     <origin xyz="0 0 0" rpy="0 0 0" />
     <geometry>
-      <mesh filename="package://robotis_op3_description/stl/ra3.stl"  scale="0.001 0.001 0.001"/>
+      <mesh filename="package://robotis_op3_description/meshes/ra3.stl"  scale="0.001 0.001 0.001"/>
     </geometry>
     <material name="Grey">
@@ -168,5 +168,5 @@
     <origin xyz="0 0 0" rpy="0 0 0" />
     <geometry>
-      <mesh filename="package://robotis_op3_description/stl/la1.stl"  scale="0.001 0.001 0.001"/>
+      <mesh filename="package://robotis_op3_description/meshes/la1.stl"  scale="0.001 0.001 0.001"/>
     </geometry>
     <material name="Grey">
@@ -178,5 +178,5 @@
     <origin xyz="0 0 0" rpy="0 0 0" />
     <geometry>
-      <mesh filename="package://robotis_op3_description/stl/la2.stl"  scale="0.001 0.001 0.001"/>
+      <mesh filename="package://robotis_op3_description/meshes/la2.stl"  scale="0.001 0.001 0.001"/>
     </geometry>
     <material name="Grey">
@@ -188,5 +188,5 @@
     <origin xyz="0 0 0" rpy="0 0 0" />
     <geometry>
-      <mesh filename="package://robotis_op3_description/stl/la3.stl"  scale="0.001 0.001 0.001"/>
+      <mesh filename="package://robotis_op3_description/meshes/la3.stl"  scale="0.001 0.001 0.001"/>
     </geometry>
     <material name="Grey">
@@ -198,5 +198,5 @@
     <origin xyz="0 0 0" rpy="0 0 0" />
     <geometry>
-      <mesh filename="package://robotis_op3_description/stl/h1.stl"  scale="0.001 0.001 0.001"/>
+      <mesh filename="package://robotis_op3_description/meshes/h1.stl"  scale="0.001 0.001 0.001"/>
     </geometry>
     <material name="Grey">
@@ -208,5 +208,5 @@
     <origin xyz="0 0 0" rpy="0 0 0" />
     <geometry>
-      <mesh filename="package://robotis_op3_description/stl/h2.stl"  scale="0.001 0.001 0.001"/>
+      <mesh filename="package://robotis_op3_description/meshes/h2.stl"  scale="0.001 0.001 0.001"/>
     </geometry>
     <material name="Grey">
