Commit message: changed package names and paths related

File: op3_description/urdf/robotis_op3.urdf.xacro (robot description, xacro)
@@ -1,15 +1,15 @@
 <?xml version="1.0" ?>
 <robot xmlns:xacro="http://ros.org/wiki/xacro" name="robotis_op3">
-  <xacro:include filename="$(find robotis_op3_description)/urdf/robotis_op3.visuals.xacro" />
-  <xacro:include filename="$(find robotis_op3_description)/urdf/robotis_op3.inertia.xacro" />
-  <xacro:include filename="$(find robotis_op3_description)/urdf/robotis_op3.structure.rleg.xacro" />
-  <xacro:include filename="$(find robotis_op3_description)/urdf/robotis_op3.structure.lleg.xacro" />
-  <xacro:include filename="$(find robotis_op3_description)/urdf/robotis_op3.structure.rarm.xacro" />
-  <xacro:include filename="$(find robotis_op3_description)/urdf/robotis_op3.structure.larm.xacro" />
-  <xacro:include filename="$(find robotis_op3_description)/urdf/robotis_op3.structure.head.xacro" />
-  <xacro:include filename="$(find robotis_op3_description)/urdf/robotis_op3.gazebo.xacro" />
-  <xacro:include filename="$(find robotis_op3_description)/urdf/robotis_op3.transmissions.xacro" />
+  <xacro:include filename="$(find op3_description)/urdf/robotis_op3.visuals.xacro" />
+  <xacro:include filename="$(find op3_description)/urdf/robotis_op3.inertia.xacro" />
+  <xacro:include filename="$(find op3_description)/urdf/robotis_op3.structure.rleg.xacro" />
+  <xacro:include filename="$(find op3_description)/urdf/robotis_op3.structure.lleg.xacro" />
+  <xacro:include filename="$(find op3_description)/urdf/robotis_op3.structure.rarm.xacro" />
+  <xacro:include filename="$(find op3_description)/urdf/robotis_op3.structure.larm.xacro" />
+  <xacro:include filename="$(find op3_description)/urdf/robotis_op3.structure.head.xacro" />
+  <xacro:include filename="$(find op3_description)/urdf/robotis_op3.gazebo.xacro" />
+  <xacro:include filename="$(find op3_description)/urdf/robotis_op3.transmissions.xacro" />
   <!--
-  <xacro:include filename="$(find robotis_op3_description)/urdf/gazebo_harness.xacro" />
+  <xacro:include filename="$(find op3_description)/urdf/gazebo_harness.xacro" />
   -->
   <!-- harness link -->

File: op3_description/urdf/robotis_op3.visuals.xacro (robot description, xacro)
@@ -8,5 +8,5 @@
     <origin xyz="0 0 0" rpy="0 0 0" />
     <geometry>
-      <mesh filename="package://robotis_op3_description/meshes/body.stl"  scale="0.001 0.001 0.001"/>
+      <mesh filename="package://op3_description/meshes/body.stl"  scale="0.001 0.001 0.001"/>
     </geometry>
     <material name="Grey">
@@ -18,5 +18,5 @@
     <origin xyz="0 0 0" rpy="0 0 0" />
     <geometry>
-      <mesh filename="package://robotis_op3_description/meshes/rl1.stl"  scale="0.001 0.001 0.001"/>
+      <mesh filename="package://op3_description/meshes/rl1.stl"  scale="0.001 0.001 0.001"/>
     </geometry>
     <material name="Grey">
@@ -28,5 +28,5 @@
     <origin xyz="0 0 0" rpy="0 0 0" />
     <geometry>
-      <mesh filename="package://robotis_op3_description/meshes/rl2.stl"  scale="0.001 0.001 0.001"/>
+      <mesh filename="package://op3_description/meshes/rl2.stl"  scale="0.001 0.001 0.001"/>
     </geometry>
     <material name="Grey">
@@ -38,5 +38,5 @@
     <origin xyz="0 0 0" rpy="0 0 0" />
     <geometry>
-      <mesh filename="package://robotis_op3_description/meshes/rl3.stl"  scale="0.001 0.001 0.001"/>
+      <mesh filename="package://op3_description/meshes/rl3.stl"  scale="0.001 0.001 0.001"/>
     </geometry>
     <material name="Grey">
@@ -48,5 +48,5 @@
     <origin xyz="0 0 0" rpy="0 0 0" />
     <geometry>
-      <mesh filename="package://robotis_op3_description/meshes/rl4.stl"  scale="0.001 0.001 0.001"/>
+      <mesh filename="package://op3_description/meshes/rl4.stl"  scale="0.001 0.001 0.001"/>
     </geometry>
     <material name="Grey">
@@ -58,5 +58,5 @@
     <origin xyz="0 0 0" rpy="0 0 0" />
     <geometry>
-      <mesh filename="package://robotis_op3_description/meshes/rl5.stl"  scale="0.001 0.001 0.001"/>
+      <mesh filename="package://op3_description/meshes/rl5.stl"  scale="0.001 0.001 0.001"/>
     </geometry>
     <material name="Grey">
@@ -68,5 +68,5 @@
     <origin xyz="0 0 0" rpy="0 0 0" />
     <geometry>
-      <mesh filename="package://robotis_op3_description/meshes/rl6.stl"  scale="0.001 0.001 0.001"/>
+      <mesh filename="package://op3_description/meshes/rl6.stl"  scale="0.001 0.001 0.001"/>
     </geometry>
     <material name="Grey">
@@ -78,5 +78,5 @@
     <origin xyz="0 0 0" rpy="0 0 0" />
     <geometry>
-      <mesh filename="package://robotis_op3_description/meshes/ll1.stl"  scale="0.001 0.001 0.001"/>
+      <mesh filename="package://op3_description/meshes/ll1.stl"  scale="0.001 0.001 0.001"/>
     </geometry>
     <material name="Grey">
@@ -88,5 +88,5 @@
     <origin xyz="0 0 0" rpy="0 0 0" />
     <geometry>
-      <mesh filename="package://robotis_op3_description/meshes/ll2.stl"  scale="0.001 0.001 0.001"/>
+      <mesh filename="package://op3_description/meshes/ll2.stl"  scale="0.001 0.001 0.001"/>
     </geometry>
     <material name="Grey">
@@ -98,5 +98,5 @@
     <origin xyz="0 0 0" rpy="0 0 0" />
     <geometry>
-      <mesh filename="package://robotis_op3_description/meshes/ll3.stl"  scale="0.001 0.001 0.001"/>
+      <mesh filename="package://op3_description/meshes/ll3.stl"  scale="0.001 0.001 0.001"/>
     </geometry>
     <material name="Grey">
@@ -108,5 +108,5 @@
     <origin xyz="0 0 0" rpy="0 0 0" />
     <geometry>
-      <mesh filename="package://robotis_op3_description/meshes/ll4.stl"  scale="0.001 0.001 0.001"/>
+      <mesh filename="package://op3_description/meshes/ll4.stl"  scale="0.001 0.001 0.001"/>
     </geometry>
     <material name="Grey">
@@ -118,5 +118,5 @@
     <origin xyz="0 0 0" rpy="0 0 0" />
     <geometry>
-      <mesh filename="package://robotis_op3_description/meshes/ll5.stl"  scale="0.001 0.001 0.001"/>
+      <mesh filename="package://op3_description/meshes/ll5.stl"  scale="0.001 0.001 0.001"/>
     </geometry>
     <material name="Grey">
@@ -128,5 +128,5 @@
     <origin xyz="0 0 0" rpy="0 0 0" />
     <geometry>
-      <mesh filename="package://robotis_op3_description/meshes/ll6.stl"  scale="0.001 0.001 0.001"/>
+      <mesh filename="package://op3_description/meshes/ll6.stl"  scale="0.001 0.001 0.001"/>
     </geometry>
     <material name="Grey">
@@ -138,5 +138,5 @@
     <origin xyz="0 0 0" rpy="0 0 0" />
     <geometry>
-      <mesh filename="package://robotis_op3_description/meshes/ra1.stl"  scale="0.001 0.001 0.001"/>
+      <mesh filename="package://op3_description/meshes/ra1.stl"  scale="0.001 0.001 0.001"/>
     </geometry>
     <material name="Grey">
@@ -148,5 +148,5 @@
     <origin xyz="0 0 0" rpy="0 0 0" />
     <geometry>
-      <mesh filename="package://robotis_op3_description/meshes/ra2.stl"  scale="0.001 0.001 0.001"/>
+      <mesh filename="package://op3_description/meshes/ra2.stl"  scale="0.001 0.001 0.001"/>
     </geometry>
     <material name="Grey">
@@ -158,5 +158,5 @@
     <origin xyz="0 0 0" rpy="0 0 0" />
     <geometry>
-      <mesh filename="package://robotis_op3_description/meshes/ra3.stl"  scale="0.001 0.001 0.001"/>
+      <mesh filename="package://op3_description/meshes/ra3.stl"  scale="0.001 0.001 0.001"/>
     </geometry>
     <material name="Grey">
@@ -168,5 +168,5 @@
     <origin xyz="0 0 0" rpy="0 0 0" />
     <geometry>
-      <mesh filename="package://robotis_op3_description/meshes/la1.stl"  scale="0.001 0.001 0.001"/>
+      <mesh filename="package://op3_description/meshes/la1.stl"  scale="0.001 0.001 0.001"/>
     </geometry>
     <material name="Grey">
@@ -178,5 +178,5 @@
     <origin xyz="0 0 0" rpy="0 0 0" />
     <geometry>
-      <mesh filename="package://robotis_op3_description/meshes/la2.stl"  scale="0.001 0.001 0.001"/>
+      <mesh filename="package://op3_description/meshes/la2.stl"  scale="0.001 0.001 0.001"/>
     </geometry>
     <material name="Grey">
@@ -188,5 +188,5 @@
     <origin xyz="0 0 0" rpy="0 0 0" />
     <geometry>
-      <mesh filename="package://robotis_op3_description/meshes/la3.stl"  scale="0.001 0.001 0.001"/>
+      <mesh filename="package://op3_description/meshes/la3.stl"  scale="0.001 0.001 0.001"/>
     </geometry>
     <material name="Grey">
@@ -198,5 +198,5 @@
     <origin xyz="0 0 0" rpy="0 0 0" />
     <geometry>
-      <mesh filename="package://robotis_op3_description/meshes/h1.stl"  scale="0.001 0.001 0.001"/>
+      <mesh filename="package://op3_description/meshes/h1.stl"  scale="0.001 0.001 0.001"/>
     </geometry>
     <material name="Grey">
@@ -208,5 +208,5 @@
     <origin xyz="0 0 0" rpy="0 0 0" />
     <geometry>
-      <mesh filename="package://robotis_op3_description/meshes/h2.stl"  scale="0.001 0.001 0.001"/>
+      <mesh filename="package://op3_description/meshes/h2.stl"  scale="0.001 0.001 0.001"/>
     </geometry>
     <material name="Grey">
