Commit message: Modified model file and launch file.

File: op3_description/urdf/robotis_op3.d435.structure.head.xacro (robot description, xacro)
@@ -69,5 +69,5 @@
   <xacro:include filename="$(find realsense2_camera)/urdf/_r430.urdf.xacro"/>
   <sensor_r430 parent="cam_link">
-    <origin xyz="0 0 0" rpy="0 0 0"/>
+    <origin xyz="0 0 0" rpy="${pi*0.5} ${-pi*0.5} 0"/>
   </sensor_r430>
   </xacro:macro>

Commit message: Fixed model file.

File: op3_description/urdf/robotis_op3.d435.structure.head.xacro (robot description, xacro)
@@ -67,8 +67,8 @@
   <link name="cam_gazebo_link">
   </link>
-  <xacro:include filename="$(find realsense2_camera)/urdf/_d430.urdf.xacro"/>
-  <sensor_r430 parent="cam_link">
-    <origin xyz="0 0 0" rpy="0 0 0"/>
-  </sensor_r430>
+  <xacro:include filename="$(find realsense2_camera)/urdf/_d435.urdf.xacro"/>
+  <sensor_d435 parent="cam_link">
+    <origin xyz="0 0 0" rpy="0 ${-pi*0.5} ${pi*0.5}"/>
+  </sensor_d435>
   </xacro:macro>
 </robot>

Commit message: Added D435 head and transforms.

File: op3_description/urdf/robotis_op3.d435.structure.head.xacro (robot description, xacro)
@@ -28,5 +28,5 @@
     </inertial>
   </link>
-  <!-- head pitch joint -->
+  <!-- head tilt joint -->
   <joint name="head_tilt" type="revolute">
     <parent link="head_pan_link"/>
@@ -38,9 +38,9 @@
   </joint>
   <xacro:insert_transmission name="head_tilt" />
-  <!-- head yaw link -->
+  <!-- head tilk link -->
   <link name="head_tilt_link">
-    <!-- <visual> -->
-    <!--   <xacro:insert_mesh_head_tilt_link /> -->
-    <!-- </visual> -->
+    <visual>
+      <xacro:insert_mesh_head_tilt_link />
+    </visual>
     <collision>
       <xacro:insert_mesh_head_tilt_link />
@@ -50,10 +50,5 @@
     </inertial>
   </link>
-  <!-- camera joint -->
-  <joint name="cam" type="fixed">
-    <origin xyz="0.01425 -0.019 0.04975" rpy="${-pi*0.5} 0 ${-pi*0.5}"/>
-    <parent link="head_tilt_link"/>
-    <child link="cam_link"/>
-  </joint>
+  <!-- camera gazebo joint -->
   <joint name="cam_gazebo" type="fixed">
     <origin xyz="0.01425 -0.019 0.04975" rpy="0 0 0"/>
@@ -61,13 +56,11 @@
     <child link="cam_gazebo_link"/>
   </joint>
-  <!-- camera link -->
-  <link name="cam_link">
-  </link>
-  <!-- camera link -->
+  <!-- camera gazebo link -->
   <link name="cam_gazebo_link">
   </link>
   <xacro:include filename="$(find realsense2_camera)/urdf/_d435.urdf.xacro"/>
-  <sensor_d435 parent="cam_link">
-    <origin xyz="0 0 0" rpy="${pi*0.5} ${-pi*0.5} 0"/>
+  <sensor_d435 parent="head_tilt_link">
+    <!-- <origin xyz="0.018 0 0.05275" rpy="${pi*0.5} ${-pi*0.5} 0"/> -->
+    <origin xyz="-0.0041 -0.019 0.04025" rpy="0 0 0"/>
   </sensor_d435>
   </xacro:macro>

File: op3_description/urdf/robotis_op3.d435.urdf.xacro (robot description, xacro)
@@ -1,5 +1,5 @@
 <?xml version="1.0" ?>
 <robot xmlns:xacro="http://ros.org/wiki/xacro" name="robotis_op3">
-  <xacro:include filename="$(find op3_description)/urdf/robotis_op3.visuals.xacro" />
+  <xacro:include filename="$(find op3_description)/urdf/robotis_op3.d435.visuals.xacro" />
   <xacro:include filename="$(find op3_description)/urdf/robotis_op3.inertia.xacro" />
   <xacro:include filename="$(find op3_description)/urdf/robotis_op3.structure.rleg.xacro" />
