Commit message: op3_description: add gz_ros2_control-system plugin and ros2_control elements
- The gazebo.xacro is missing the ros2_control system. This prevents the op3_gazebo_ros2 simulation package from working.
- Added from https://github.com/Jay-Song/op3_gazebo_ros2/blob/main/gazebo/robotis_op3.gazebo.xacro

Signed-off-by: Rhys Mainwaring <rhys.mainwaring@me.com>

File: op3_description/urdf/robotis_op3.gazebo.xacro (robot description, xacro)
@@ -164,4 +164,240 @@
       </plugin>
     </gazebo>
+    <!-- For Gazebo Control and Sensors -->
+    <gazebo>
+      <plugin filename="gz_ros2_control-system" name="gz_ros2_control::GazeboSimROS2ControlPlugin">
+        <parameters>$(find op3_gazebo_ros2)/config/robotis_op3_gazebo_config.yaml</parameters>
+      </plugin>
+      <plugin filename="gz-sim-sensors-system" name="gz::sim::systems::Sensors">
+        <render_engine>ogre2</render_engine>
+      </plugin>
+      <plugin filename="gz-sim-imu-system" name="gz::sim::systems::Imu"/>
+    </gazebo>
+    <!-- For Ros2 Control -->
+    <ros2_control name="GazeboSimSystem" type="system">
+      <hardware>
+        <plugin>gz_ros2_control/GazeboSimSystem</plugin>
+      </hardware>
+      <joint name="r_sho_pitch">
+        <command_interface name="position">
+          <param name="min">-3.14</param>
+          <param name="max">3.14</param>
+        </command_interface>
+        <state_interface name="position">
+          <param name="initial_value">0.0</param>
+        </state_interface>
+        <state_interface name="velocity"/>
+        <state_interface name="effort"/>
+      </joint>
+      <joint name="l_sho_pitch">
+        <command_interface name="position">
+          <param name="min">-3.14</param>
+          <param name="max">3.14</param>
+        </command_interface>
+        <state_interface name="position">
+          <param name="initial_value">0.0</param>
+        </state_interface>
+        <state_interface name="velocity"/>
+        <state_interface name="effort"/>
+      </joint>
+      <joint name="r_sho_roll">
+        <command_interface name="position">
+          <param name="min">-3.14</param>
+          <param name="max">3.14</param>
+        </command_interface>
+        <state_interface name="position">
+          <param name="initial_value">0.0</param>
+        </state_interface>
+        <state_interface name="velocity"/>
+        <state_interface name="effort"/>
+      </joint>
+      <joint name="l_sho_roll">
+        <command_interface name="position">
+          <param name="min">-3.14</param>
+          <param name="max">3.14</param>
+        </command_interface>
+        <state_interface name="position">
+          <param name="initial_value">0.0</param>
+        </state_interface>
+        <state_interface name="velocity"/>
+        <state_interface name="effort"/>
+      </joint>
+      <joint name="r_el">
+        <command_interface name="position">
+          <param name="min">-3.14</param>
+          <param name="max">3.14</param>
+        </command_interface>
+        <state_interface name="position">
+          <param name="initial_value">0.0</param>
+        </state_interface>
+        <state_interface name="velocity"/>
+        <state_interface name="effort"/>
+      </joint>
+      <joint name="l_el">
+        <command_interface name="position">
+          <param name="min">-3.14</param>
+          <param name="max">3.14</param>
+        </command_interface>
+        <state_interface name="position">
+          <param name="initial_value">0.0</param>
+        </state_interface>
+        <state_interface name="velocity"/>
+        <state_interface name="effort"/>
+      </joint>
+      <joint name="r_hip_yaw">
+        <command_interface name="position">
+          <param name="min">-3.14</param>
+          <param name="max">3.14</param>
+        </command_interface>
+        <state_interface name="position">
+          <param name="initial_value">0.0</param>
+        </state_interface>
+        <state_interface name="velocity"/>
+        <state_interface name="effort"/>
+      </joint>
+      <joint name="l_hip_yaw">
+        <command_interface name="position">
+          <param name="min">-3.14</param>
+          <param name="max">3.14</param>
+        </command_interface>
+        <state_interface name="position">
+          <param name="initial_value">0.0</param>
+        </state_interface>
+        <state_interface name="velocity"/>
+        <state_interface name="effort"/>
+      </joint>
+      <joint name="r_hip_roll">
+        <command_interface name="position">
+          <param name="min">-3.14</param>
+          <param name="max">3.14</param>
+        </command_interface>
+        <state_interface name="position">
+          <param name="initial_value">0.0</param>
+        </state_interface>
+        <state_interface name="velocity"/>
+        <state_interface name="effort"/>
+      </joint>
+      <joint name="l_hip_roll">
+        <command_interface name="position">
+          <param name="min">-3.14</param>
+          <param name="max">3.14</param>
+        </command_interface>
+        <state_interface name="position">
+          <param name="initial_value">0.0</param>
+        </state_interface>
+        <state_interface name="velocity"/>
+        <state_interface name="effort"/>
+      </joint>
+      <joint name="r_hip_pitch">
+        <command_interface name="position">
+          <param name="min">-3.14</param>
+          <param name="max">3.14</param>
+        </command_interface>
+        <state_interface name="position">
+          <param name="initial_value">0.0</param>
+        </state_interface>
+        <state_interface name="velocity"/>
+        <state_interface name="effort"/>
+      </joint>
+      <joint name="l_hip_pitch">
+        <command_interface name="position">
+          <param name="min">-3.14</param>
+          <param name="max">3.14</param>
+        </command_interface>
+        <state_interface name="position">
+          <param name="initial_value">0.0</param>
+        </state_interface>
+        <state_interface name="velocity"/>
+        <state_interface name="effort"/>
+      </joint>
+      <joint name="r_knee">
+        <command_interface name="position">
+          <param name="min">-3.14</param>
+          <param name="max">3.14</param>
+        </command_interface>
+        <state_interface name="position">
+          <param name="initial_value">0.0</param>
+        </state_interface>
+        <state_interface name="velocity"/>
+        <state_interface name="effort"/>
+      </joint>
+      <joint name="l_knee">
+        <command_interface name="position">
+          <param name="min">-3.14</param>
+          <param name="max">3.14</param>
+        </command_interface>
+        <state_interface name="position">
+          <param name="initial_value">0.0</param>
+        </state_interface>
+        <state_interface name="velocity"/>
+        <state_interface name="effort"/>
+      </joint>
+      <joint name="r_ank_pitch">
+        <command_interface name="position">
+          <param name="min">-3.14</param>
+          <param name="max">3.14</param>
+        </command_interface>
+        <state_interface name="position">
+          <param name="initial_value">0.0</param>
+        </state_interface>
+        <state_interface name="velocity"/>
+        <state_interface name="effort"/>
+      </joint>
+      <joint name="l_ank_pitch">
+        <command_interface name="position">
+          <param name="min">-3.14</param>
+          <param name="max">3.14</param>
+        </command_interface>
+        <state_interface name="position">
+          <param name="initial_value">0.0</param>
+        </state_interface>
+        <state_interface name="velocity"/>
+        <state_interface name="effort"/>
+      </joint>
+      <joint name="r_ank_roll">
+        <command_interface name="position">
+          <param name="min">-3.14</param>
+          <param name="max">3.14</param>
+        </command_interface>
+        <state_interface name="position">
+          <param name="initial_value">0.0</param>
+        </state_interface>
+        <state_interface name="velocity"/>
+        <state_interface name="effort"/>
+      </joint>
+      <joint name="l_ank_roll">
+        <command_interface name="position">
+          <param name="min">-3.14</param>
+          <param name="max">3.14</param>
+        </command_interface>
+        <state_interface name="position">
+          <param name="initial_value">0.0</param>
+        </state_interface>
+        <state_interface name="velocity"/>
+        <state_interface name="effort"/>
+      </joint>
+      <joint name="head_pan">
+        <command_interface name="position">
+          <param name="min">-3.14</param>
+          <param name="max">3.14</param>
+        </command_interface>
+        <state_interface name="position">
+          <param name="initial_value">0.0</param>
+        </state_interface>
+        <state_interface name="velocity"/>
+        <state_interface name="effort"/>
+      </joint>
+      <joint name="head_tilt">
+        <command_interface name="position">
+          <param name="min">-3.14</param>
+          <param name="max">3.14</param>
+        </command_interface>
+        <state_interface name="position">
+          <param name="initial_value">0.0</param>
+        </state_interface>
+        <state_interface name="velocity"/>
+        <state_interface name="effort"/>
+      </joint>
+    </ros2_control>
     <gazebo reference="cam_gazebo_link">
       <sensor name='camera' type='camera'>

Commit message: op3_description: remove unsupported material type from gazebo.xacro
- Material scripts are not supported in later versions of Gazebo.

Signed-off-by: Rhys Mainwaring <rhys.mainwaring@me.com>

File: op3_description/urdf/robotis_op3.gazebo.xacro (robot description, xacro)
@@ -5,5 +5,4 @@
       <mu1>0.2</mu1>
       <mu2>0.2</mu2>
-      <material>Gazebo/White</material>
       <selfCollide>false</selfCollide>
     </gazebo>
@@ -12,5 +11,4 @@
       <mu1>0.2</mu1>
       <mu2>0.2</mu2>
-      <material>Gazebo/White</material>
       <selfCollide>false</selfCollide>
     </gazebo>
@@ -18,5 +16,4 @@
       <mu1>0.2</mu1>
       <mu2>0.2</mu2>
-      <material>Gazebo/White</material>
       <selfCollide>false</selfCollide>
     </gazebo>
@@ -24,5 +21,4 @@
       <mu1>0.2</mu1>
       <mu2>0.2</mu2>
-      <material>Gazebo/White</material>
       <selfCollide>false</selfCollide>
     </gazebo>
@@ -30,5 +26,4 @@
       <mu1>0.2</mu1>
       <mu2>0.2</mu2>
-      <material>Gazebo/White</material>
       <selfCollide>false</selfCollide>
     </gazebo>
@@ -36,5 +31,4 @@
       <mu1>0.2</mu1>
       <mu2>0.2</mu2>
-      <material>Gazebo/White</material>
       <selfCollide>false</selfCollide>
     </gazebo>
@@ -47,5 +41,4 @@
       <maxVel>1.0</maxVel>
       <minDepth>0.001</minDepth>
-      <material>Gazebo/White</material>
     </gazebo>
     <!-- right leg links -->
@@ -53,5 +46,4 @@
       <mu1>0.2</mu1>
       <mu2>0.2</mu2>
-      <material>Gazebo/White</material>
       <selfCollide>false</selfCollide>
     </gazebo>
@@ -59,5 +51,4 @@
       <mu1>0.2</mu1>
       <mu2>0.2</mu2>
-      <material>Gazebo/White</material>
       <selfCollide>false</selfCollide>
     </gazebo>
@@ -65,5 +56,4 @@
       <mu1>0.2</mu1>
       <mu2>0.2</mu2>
-      <material>Gazebo/White</material>
       <selfCollide>false</selfCollide>
     </gazebo>
@@ -71,5 +61,4 @@
       <mu1>0.2</mu1>
       <mu2>0.2</mu2>
-      <material>Gazebo/White</material>
       <selfCollide>false</selfCollide>
     </gazebo>
@@ -77,5 +66,4 @@
       <mu1>0.2</mu1>
       <mu2>0.2</mu2>
-      <material>Gazebo/White</material>
       <selfCollide>false</selfCollide>
     </gazebo>
@@ -89,10 +77,8 @@
       <maxVel>1.0</maxVel>
       <minDepth>0.001</minDepth>
-      <material>Gazebo/White</material>
     </gazebo>
     <gazebo reference="r_sho_pitch_link">
       <mu1>0.2</mu1>
       <mu2>0.2</mu2>
-      <material>Gazebo/White</material>
       <selfCollide>false</selfCollide>
     </gazebo>
@@ -100,5 +86,4 @@
       <mu1>0.2</mu1>
       <mu2>0.2</mu2>
-      <material>Gazebo/White</material>
       <selfCollide>false</selfCollide>
     </gazebo>
@@ -106,5 +91,4 @@
       <mu1>0.2</mu1>
       <mu2>0.2</mu2>
-      <material>Gazebo/White</material>
       <selfCollide>false</selfCollide>
     </gazebo>
@@ -112,5 +96,4 @@
       <mu1>0.2</mu1>
       <mu2>0.2</mu2>
-      <material>Gazebo/White</material>
       <selfCollide>false</selfCollide>
     </gazebo>
@@ -118,5 +101,4 @@
       <mu1>0.2</mu1>
       <mu2>0.2</mu2>
-      <material>Gazebo/White</material>
       <selfCollide>false</selfCollide>
     </gazebo>
@@ -124,5 +106,4 @@
       <mu1>0.2</mu1>
       <mu2>0.2</mu2>
-      <material>Gazebo/White</material>
       <selfCollide>false</selfCollide>
     </gazebo>
@@ -130,5 +111,4 @@
       <mu1>0.2</mu1>
       <mu2>0.2</mu2>
-      <material>Gazebo/White</material>
       <selfCollide>false</selfCollide>
     </gazebo>
@@ -136,5 +116,4 @@
       <mu1>0.2</mu1>
       <mu2>0.2</mu2>
-      <material>Gazebo/White</material>
       <selfCollide>false</selfCollide>
     </gazebo>

Commit message: op3_description: add xacro parameter for Gazebo controllers param file
Signed-off-by: Rhys Mainwaring <rhys.mainwaring@me.com>

File: op3_description/urdf/robotis_op3.gazebo.xacro (robot description, xacro)
@@ -1,5 +1,5 @@
 <?xml version="1.0"?>
 <robot xmlns:xacro="http://ros.org/wiki/xacro">
-  <xacro:macro name="robotis_op3_gazebo">
+  <xacro:macro name="robotis_op3_gazebo" params="gazebo_controllers_param_file">
     <gazebo reference="body_link">
       <mu1>0.2</mu1>
@@ -146,5 +146,5 @@
     <gazebo>
       <plugin filename="gz_ros2_control-system" name="gz_ros2_control::GazeboSimROS2ControlPlugin">
-        <parameters>$(find op3_gazebo_ros2)/config/robotis_op3_gazebo_config.yaml</parameters>
+        <parameters>${gazebo_controllers_param_file}</parameters>
       </plugin>
       <plugin filename="gz-sim-sensors-system" name="gz::sim::systems::Sensors">
